File: hardware/KungFuSID.kicad_sch (KiCad schematic)
At the start: 33 parts, among them J1 SWD, U1 AMS1117-3.3, U2 C64-SID-Socket-hackup, U3 GD32F405RGT6, U4 LM321, Y1 8MHz

Commit message: Attempts to make Potxy(please still use release version) Update of hardware files
Parts:
- added R11, R12: 470, Resistor_SMD:R_0402_1005Metric, symbol KungFuSID-rescue:R-Device
Connections:
- net POT_X: now also R11.1; no longer U2.24 (POT_X)
- net POT_Y: now also R12.1; no longer U2.23 (POT_Y)
- new net I_P_X: R11.2, U2.24 (POT_X)
- new net I_P_Y: R12.2, U2.23 (POT_Y)
